File: Adafruit tftcaptouchshield rev C.brd (EAGLE design)
At the start: 70.4 x 54.4 mm, 36 parts, among them IC4 MIC5225-3.3, IC5 AXP803, Q1 MMBT2222, SW1 SPST_TACT-EVQQ2, U2 STMPE610, U3 74HC4050

Commit message: Updated to latest versions
Parts:
- removed ICSP_SI1, PIN3: (no value), microbuilder:SOLDERJUMPER_REFLOW_NOPASTE
- removed Q1: MMBT2222, transistor-neu-to92:SOT23-BEC
- removed R5: 1K, rcl:R0805
- removed R7: 10K, rcl:R0805
- removed U2: STMPE610, microbuilder:QFN16_3MM
- added D5, D7: (no value), microbuilder:SOLDERJUMPER_ARROW_NOPASTE
- added Q2, Q3, Q4: BSS138, microbuilder:SOT23-WIDE
- added R13, R14, R15, R16: 10K, microbuilder:0805-NO
- added SCL_A5, SDA_A4: (no value), microbuilder:SOLDERJUMPER_REFLOW_NOPASTE
- added SJ4: (no value), microbuilder:SOLDERJUMPER_2WAY_OPEN_NOPASTE
- added U$7: (no value), microbuilder:PCBFEAT-REV-040
- C1, C2, C3, C4, C5: device adafruit:C0805K -> microbuilder:0805-NO
- ICSP_CLK, ICSP_SI, ICSP_SO: device microbuilder:SOLDERJUMPER_REFLOW_NOPASTE -> microbuilder:SOLDERJUMPER_CLOSEDWIRE
- R1, R2, R3, R4, R6, R8: device rcl:R0805 -> microbuilder:0805-NO
- R9: value 1K -> 2.2K; device rcl:R0805 -> microbuilder:0805-NO
- SJ1, SJ2, SJ3: device microbuilder:SOLDERJUMPER_CLOSEDWIRE -> microbuilder:SOLDERJUMPER_ARROW_NOPASTE
- U$10, U$11, U$19: value FIDUCIAL -> FIDUCIAL_1MM; device adafruit:FIDUCIAL_1MM -> microbuilder:FIDUCIAL_1MM
- U$2: value DISP_LCD_1.28IN_240X320_50PIN -> 2.8" TFT + CTP
- moved U$10 13.0 mm to (53.7, 44.2)
- moved U$20 4.19 mm to (0.25, 12.8)
- moved ICSP_SI 4.15 mm to (67.2, 19.4)
- moved ICSP_SO 4.15 mm to (64.9, 19.4)
- moved ICSP_CLK 4.15 mm to (62.6, 19.4)
- moved SJ1 4.09 mm to (67.2, 13.5)
- moved SJ2 4.09 mm to (64.9, 13.5)
- moved SJ3 4.09 mm to (62.6, 13.5)
Connections:
- net CARDCS_5V renamed CARDCS
- net MOSI_5V renamed MOSI
- net N$8 renamed !RESET
- net SCLK_5V renamed SCLK
- net TFT_CS_5V renamed TFT_CS
- net TFT_DC_5V renamed TFT_DC
- removed net N$16: Q1.B, R5.2
- removed net N$5: PIN3.1, R5.1, R9.1
- removed net N$7: PIN3.2, U$17.D3
- removed net RT_CS_3V: U2.5, U3.15
- removed net RT_CS_5V: R7.1, U$17.D8, U3.14
- removed net TS_INT: ICSP_SI1.1, U2.2
- removed net VCC: C1.1, C2.1, C3.1, C4.1, IC4.5, IC5.3, R6.2, R7.2, R8.2, U$2.40, U$2.41, U$2.42, U$2.7, U$2.8, U$2.9, U$3.4, U2.14, U2.6, U2.9, U3.1
- removed net XL: U$2.46, U2.16
- removed net XR: U$2.44, U2.13
- removed net YD: U$2.45, U2.15
- removed net YU: U$2.47, U2.1
- new net 3.3V: C1.1, C2.1, C3.1, C4.1, IC4.5, IC5.3, Q2.1, Q3.1, R15.1, R16.2, R6.2, SJ4.1, U$2.40, U$2.41, U$2.42, U$2.7, U$2.8, U$2.9, U$3.4, U3.1
- new net BACKLITE: D5.2, Q4.1, R9.1
- new net D5: D5.1, U$17.D5
- new net N$17: SDA_A4.1, U$17.A4
- new net N$18: SCL_A5.1, U$17.A5
- new net SCL: Q2.3, R13.1, SCL_A5.2, U$17.SCL
- new net SCL_3V: Q2.2, R16.1, U$2.44
- new net SDA: Q3.3, R14.2, SDA_A4.2, U$17.SDA
- new net SDA_3V: Q3.2, R15.2, U$2.45
- new net TP_IRQ: D7.1, U$2.46
- new net VCCIO: R13.2, R14.1, R8.2, R9.2, SJ4.2, U$17.IOREF
- net +5V: now also SJ4.3; no longer R9.2
- net D7: now also D7.2; no longer ICSP_SI1.2
- net GND: now also Q4.2; no longer Q1.E, U2.10
- net MISO: no longer U2.3
- net MOSI_3V: no longer U2.7
- net N$1: now also Q4.3; no longer Q1.C
- net SCLK_3V: no longer U2.4
- net TFT_RST: now also U$2.47
Routing:
- net 3.3V: track 0.00 -> 191.2 mm, vias 0 -> 5
- net VCC: track 157.1 -> 0.00 mm, vias 7 -> 0
- net SCL: track 0.00 -> 137.7 mm, vias 0 -> 3
- net SDA: track 0.00 -> 131.3 mm, vias 0 -> 2
- net VCCIO: track 0.00 -> 103.5 mm, vias 0 -> 3
- net TP_IRQ: track 0.00 -> 64.3 mm, vias 0 -> 2
- net TS_INT: track 62.6 -> 0.00 mm, vias 2 -> 0
- net SDA_3V: track 0.00 -> 56.3 mm, vias 0 -> 2
- net SCL_3V: track 0.00 -> 54.7 mm, vias 0 -> 2
- net RT_CS_5V: track 42.7 -> 0.00 mm, vias 2 -> 0
- net N$5: track 29.5 -> 0.00 mm
- net BACKLITE: track 0.00 -> 26.1 mm
- net SCLK: track 83.3 -> 106.1 mm
- net +5V: track 83.2 -> 100.5 mm
- net N$17: track 0.00 -> 10.5 mm
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- added copper zone on layer 16, net GND
Other:
- outline, holes or cut-outs redrawn
- board text added: "#5"
- board text added: "3V"
- board text added: "5V"
- board text added: "D11/12/D13 SPI (old Ard)"
- board text added: "Default SPI ICSP"
- board text added: "I2C jumpers for <R3"
- board text added: "IOREF"
- board text added: "SCL"
- board text added: "SDA"
- board text added: "TFT CS #10 TFT DC #9 Card CS #4"
- board text added: "TFT: ILI9341 SPI TS: FT6206 I2C"
- board text added: "and microSD"
- board text added: "w/Cap Touch"
- board text removed: "#3"
- board text removed: "ICSP"
- board text removed: "Leo/Mega use ICSP & cut 11-13"
- board text removed: "TFT CS #10 TFT DC #9 TS CS #8 Card CS #4"
- board text removed: "TFT: ILI9341 SPI TS: STMPE610 SPI"
- board text removed: "and microSD card"
- board text removed: "v2.0"
- board text removed: "w/Touchscreen"
